Commit message: succ

File: install/diff_control/share/diff_control/ros2_control/diffbot_model_our.urdf.xacro (robot description, xacro)
@@ -4,5 +4,5 @@
   <xacro:property name="base_width" value="0.44"/>
   <xacro:property name="base_length" value="0.34"/>
-  <xacro:property name="base_height" value="0.3"/>
+  <xacro:property name="base_height" value="0.32"/>
   <xacro:property name="wheel_radius" value="0.08"/>
   <xacro:property name="wheel_width" value="0.03"/>
@@ -118,8 +118,8 @@
     <xacro:caster prefix="left_caster" x_reflect="1" y_reflect="1" />
     <xacro:caster prefix="right_caster" x_reflect="1" y_reflect="-1" /> -->
-    <link name="front_caster">
+    <link name="left_front_caster">
       <visual>
         <geometry>
-          <sphere radius="${(wheel_radius+wheel_zoff-(base_height/2))}"/>
+          <sphere radius="${(wheel_radius + wheel_zoff - (base_height / 2))}"/>
         </geometry>
         <material name="Cyan">
@@ -130,43 +130,40 @@
         <origin xyz="0 0 0" rpy="0 0 0"/>
         <geometry>
-          <sphere radius="${(wheel_radius+wheel_zoff-(base_height/2))}"/>
+          <sphere radius="${(wheel_radius + wheel_zoff - (base_height / 2))}"/>
         </geometry>
       </collision>
-      <xacro:sphere_inertia m="0.5" r="${(wheel_radius+wheel_zoff-(base_height/2))}"/>
+      <xacro:sphere_inertia m="0.5" r="${(wheel_radius + wheel_zoff - (base_height / 2))}"/>
     </link>
-    <joint name="caster_joint" type="fixed">
-      <parent link="base_link"/>
-      <child link="front_caster"/>
-      <origin xyz="${caster_xoff} 0.0 ${-(base_height/2)}" rpy="0 0 0"/>
-    </joint>
-  <!-- Small wheels -->
-  <!-- <xacro:macro name="caster" params="prefix y_reflect">
-    <link name="${prefix}_link">
+    <!-- 右前万向轮 -->
+    <link name="right_front_caster">
       <visual>
-        <origin xyz="0 0 0" rpy="${pi/2} 0 0"/>
-        <geometry>
-            <cylinder radius="0.02" length="${wheel_width}"/>
-        </geometry>
-        <material name="Gray">
-          <color rgba="0.5 0.5 0.5 1.0"/>
+        <geometry>
+          <sphere radius="${(wheel_radius + wheel_zoff - (base_height / 2))}"/>
+        </geometry>
+        <material name="Cyan">
+          <color rgba="0 1.0 1.0 1.0"/>
         </material>
       </visual>
       <collision>
-        <origin xyz="0 0 0" rpy="${pi/2} 0 0"/>
-        <geometry>
-          <cylinder radius="0.02" length="${wheel_width}"/>
+        <origin xyz="0 0 0" rpy="0 0 0"/>
+        <geometry>
+          <sphere radius="${(wheel_radius + wheel_zoff - (base_height / 2))}"/>
         </geometry>
       </collision>
-      <xacro:cylinder_inertia m="3.5" r="0.02" h="${wheel_width}"/>
+      <xacro:sphere_inertia m="0.5" r="${(wheel_radius + wheel_zoff - (base_height / 2))}"/>
     </link>
-    <joint name="${prefix}_joint" type="continuous">
+    <!-- 前万向轮关节 -->
+    <joint name="left_front_caster_joint" type="fixed">
       <parent link="base_link"/>
-      <child link="${prefix}_link"/>
-      <origin xyz="0.25 ${y_reflect*0.18} -0.235" rpy="0 0 0"/>
-      <axis xyz="0 1 0"/>
+      <child link="left_front_caster"/>
+      <origin xyz="${caster_xoff} ${base_width / 2 - wheel_ygap} ${-(base_height / 2)}" rpy="0 0 0"/>
+      <axis xyz="0 1 0"/>  <!-- 旋转轴 -->
     </joint>
-  </xacro:macro>
-  <xacro:caster prefix="caster_l" y_reflect="1" />
-  <xacro:caster prefix="caster_r" y_reflect="-1" /> -->
+    <joint name="right_front_caster_joint" type="fixed">
+      <parent link="base_link"/>
+      <child link="right_front_caster"/>
+      <origin xyz="${caster_xoff} ${-(base_width / 2 - wheel_ygap)} ${-(base_height / 2)}" rpy="0 0 0"/>
+      <axis xyz="0 1 0"/>  <!-- 旋转轴 -->
+    </joint>
   <link name="imu_link">
     <visual>
@@ -185,5 +182,5 @@
     <parent link="base_link"/>
     <child link="imu_link"/>
-    <origin xyz="0.13 0 -0.12"/>
+    <origin xyz="0 0 0.17" rpy="0 0 0"/>
   </joint>
   <gazebo reference="imu_link">
@@ -276,5 +273,5 @@
     <parent link="base_link"/>
     <child link="lidar_link"/>
-    <origin xyz="0.245 0 0.19" rpy="0 0 0"/>
+    <origin xyz="0 0 0.285" rpy="0 0 0"/>
   </joint>
   <gazebo reference="lidar_link">
@@ -312,21 +309,141 @@
     </sensor>
   </gazebo>
-  <link name="camera_link">
-    <visual>
-      <geometry>
-        <box size="0.05 0.05 0.02"/>
-      </geometry>
-    </visual>
-    <collision>
-      <geometry>
-        <box size="0.05 0.05 0.02"/>
-      </geometry>
-    </collision>
-    <xacro:box_inertia m="0.05" w="0.05" d="0.05" h="0.02"/>
-  </link>
-  <joint name="camera_joint" type="fixed">
-    <parent link="base_link"/>
-    <child link="camera_link"/>
-    <origin xyz="0.13 0 -0.12"/>
+  <!-- Camera Front -->
+  <link name="CAM_FRONT">
+    <visual>
+      <geometry>
+        <box size="0.05 0.05 0.02"/>
+      </geometry>
+      <material name="black"/>
+    </visual>
+    <collision>
+      <geometry>
+        <box size="0.05 0.05 0.02"/>
+      </geometry>
+    </collision>
+    <inertial>
+      <mass value="0.05"/>
+      <inertia ixx="0.0001" ixy="0.0" ixz="0.0" iyy="0.0001" iyz="0.0" izz="0.0001"/>
+    </inertial>
+  </link>
+  <joint name="CAM_FRONT_joint" type="fixed">
+    <parent link="base_link"/>
+    <child link="CAM_FRONT"/>
+    <origin xyz="0.17 0.0 0.185" rpy="0 0 0"/> <!-- 0° -->
+  </joint>
+  <!-- Camera Front Right -->
+  <link name="CAM_FRONT_LEFT">
+    <visual>
+      <geometry>
+        <box size="0.05 0.05 0.02"/>
+      </geometry>
+      <material name="black"/>
+    </visual>
+    <collision>
+      <geometry>
+        <box size="0.05 0.05 0.02"/>
+      </geometry>
+    </collision>
+    <inertial>
+      <mass value="0.05"/>
+      <inertia ixx="0.0001" ixy="0.0" ixz="0.0" iyy="0.0001" iyz="0.0" izz="0.0001"/>
+    </inertial>
+  </link>
+  <joint name="CAM_FRONT_LEFT_joint" type="fixed">
+    <parent link="base_link"/>
+    <child link="CAM_FRONT_LEFT"/>
+    <origin xyz="0.12 0.22 0.185" rpy="0 0 1.0472"/> <!-- 60° -->
+  </joint>
+  <!-- Camera Back Right -->
+  <link name="CAM_BACK_LEFT">
+    <visual>
+      <geometry>
+        <box size="0.05 0.05 0.02"/>
+      </geometry>
+      <material name="black"/>
+    </visual>
+    <collision>
+      <geometry>
+        <box size="0.05 0.05 0.02"/>
+      </geometry>
+    </collision>
+    <inertial>
+      <mass value="0.05"/>
+      <inertia ixx="0.0001" ixy="0.0" ixz="0.0" iyy="0.0001" iyz="0.0" izz="0.0001"/>
+    </inertial>
+  </link>
+  <joint name="CAM_BACK_LEFT_joint" type="fixed">
+    <parent link="base_link"/>
+    <child link="CAM_BACK_LEFT"/>
+    <origin xyz="-0.12 0.22 0.185" rpy="0 0 2.0944"/> <!-- 120° -->
+  </joint>
+  <!-- Camera Back -->
+  <link name="CAM_BACK">
+    <visual>
+      <geometry>
+        <box size="0.05 0.05 0.02"/>
+      </geometry>
+      <material name="black"/>
+    </visual>
+    <collision>
+      <geometry>
+        <box size="0.05 0.05 0.02"/>
+      </geometry>
+    </collision>
+    <inertial>
+      <mass value="0.05"/>
+      <inertia ixx="0.0001" ixy="0.0" ixz="0.0" iyy="0.0001" iyz="0.0" izz="0.0001"/>
+    </inertial>
+  </link>
+  <joint name="CAM_BACK_joint" type="fixed">
+    <parent link="base_link"/>
+    <child link="CAM_BACK"/>
+    <origin xyz="-0.17 0.0 0.185" rpy="0 0 3.1416"/> <!-- 180° -->
+  </joint>
+  <!-- Camera Back Left -->
+  <link name="CAM_BACK_RIGHT">
+    <visual>
+      <geometry>
+        <box size="0.05 0.05 0.02"/>
+      </geometry>
+      <material name="black"/>
+    </visual>
+    <collision>
+      <geometry>
+        <box size="0.05 0.05 0.02"/>
+      </geometry>
+    </collision>
+    <inertial>
+      <mass value="0.05"/>
+      <inertia ixx="0.0001" ixy="0.0" ixz="0.0" iyy="0.0001" iyz="0.0" izz="0.0001"/>
+    </inertial>
+  </link>
+  <joint name="CAM_BACK_RIGHT_joint" type="fixed">
+    <parent link="base_link"/>
+    <child link="CAM_BACK_RIGHT"/>
+    <origin xyz="-0.12 -0.22 0.185" rpy="0 0 -2.0944"/> <!-- 240° -->
+  </joint>
+  <!-- Camera Front Left -->
+  <link name="CAM_FRONT_RIGHT">
+    <visual>
+      <geometry>
+        <box size="0.05 0.05 0.02"/>
+      </geometry>
+      <material name="black"/>
+    </visual>
+    <collision>
+      <geometry>
+        <box size="0.05 0.05 0.02"/>
+      </geometry>
+    </collision>
+    <inertial>
+      <mass value="0.05"/>
+      <inertia ixx="0.0001" ixy="0.0" ixz="0.0" iyy="0.0001" iyz="0.0" izz="0.0001"/>
+    </inertial>
+  </link>
+  <joint name="CAM_FRONT_RIGHT_joint" type="fixed">
+    <parent link="base_link"/>
+    <child link="CAM_FRONT_RIGHT"/>
+    <origin xyz="0.12 -0.22 0.185" rpy="0 0 -1.0472"/> <!-- 300° -->
   </joint>
 </robot>
